Commit message: Fixed Inertia Tensors and Colors

File: src/urdf/restorebot.urdf.xacro (robot description, xacro)
@@ -22,11 +22,11 @@
 	</xacro:macro>
 	<material name="blue">
-	<color rgba="0 0 0.8 1"/>
+		<color rgba="0 0 0.8 1"/>
 	</material>
 	<material name="black">
-	<color rgba="0 0 0 1"/>
+		<color rgba="0 0 0 1"/>
 	</material>
 	<material name="white">
-	<color rgba="1 1 1 1"/>
+			<color rgba="1 1 1 1"/>
 	</material>
 	<link name="platform_base">
@@ -38,4 +38,5 @@
 		<visual>
 			<xacro:platform_geom />
+			<material name = "black"/>
 		</visual>
 		<collision>
@@ -60,4 +61,5 @@
 			<xacro:armLink1_geom />
 			<xacro:armLink1_offset />
+			<material name="white"/>
 		</visual>
 		<collision>
@@ -67,5 +69,5 @@
 		<inertial>
 			<mass value="${armLink1Mass}" />
-			<inertia ixx="1.0" ixy="0.0" ixz="0.0" iyy="1.0" iyz="0.0" izz="1.0" />
+			<inertia ixx="${armLink1Len^2/3+armLink1Rad^2/4}" ixy="0.0" ixz="0.0" iyy="${armLink1Len^2/3+armLink1Rad^2/4}" iyz="0.0" izz="${armLink1Rad^2/2}" />
 		</inertial>
 	</link>
@@ -90,4 +92,5 @@
 			<xacro:armLink1square_geom />
 			<xacro:armLink1square_offset />
+			<material name="white"/>
 		</visual>
 		<collision>
@@ -97,7 +100,8 @@
 		<inertial>
 			<mass value="${armLink1squareMass}" />
-			<inertia ixx="1.0" ixy="0.0" ixz="0.0" iyy="1.0" iyz="0.0" izz="1.0" />
-		</inertial>
-	</link>
+			<inertia ixx="${armLink1squareLen^2 * 5/12}" ixy="0.0" ixz="0.0" iyy="${armLink1squareLen^2 * 5/12}" iyz="0.0" izz="${armLink1squareLen^2 / 6}" />
+		</inertial>
+	</link>
+s
 	<joint name="armLink1Fixed" type ="fixed">
 		<parent link="armLink1"/>
@@ -119,4 +123,5 @@
 			<xacro:armLink2_geom />
 			<xacro:armLink2_offset />
+			<material name="blue"/>
 		</visual>
 		<collision>
@@ -126,5 +131,5 @@
 		<inertial>
 			<mass value="${armLink2Mass}" />
-			<inertia ixx="1.0" ixy="0.0" ixz="0.0" iyy="1.0" iyz="0.0" izz="1.0" />
+			<inertia ixx="${armLink2Len^2 /6}" ixy="0.0" ixz="0.0" iyy="${armLink2Len^2/6}" iyz="0.0" izz="${armLink2Len^2 /6}" />
 		</inertial>
 	</link>
@@ -151,4 +156,5 @@
 			<xacro:armLink3_geom />
 			<xacro:armLink3_offset />
+			<material name="white"/>
 		</visual>
 		<collision>
@@ -158,5 +164,5 @@
 		<inertial>
 			<mass value="${armLink3Mass}" />
-			<inertia ixx="1.0" ixy="0.0" ixz="0.0" iyy="1.0" iyz="0.0" izz="1.0" />
+			<inertia ixx="${armLink3Len^2/3+armLink3Rad^2/4}" ixy="0.0" ixz="0.0" iyy="${armLink3Len^2/3+armLink3Rad^2/4}" iyz="0.0" izz="${armLink3Rad^2/2}" />
 		</inertial>
 	</link>
@@ -181,4 +187,5 @@
 			<xacro:armLink3square_geom />
 			<xacro:armLink3square_offset />
+			<material name="white"/>
 		</visual>
 		<collision>
@@ -188,5 +195,5 @@
 		<inertial>
 			<mass value="${armLink3squareMass}" />
-			<inertia ixx="1.0" ixy="0.0" ixz="0.0" iyy="1.0" iyz="0.0" izz="1.0" />
+			<inertia ixx="${armLink3squareLen^2 * 5/12}" ixy="0.0" ixz="0.0" iyy="${armLink3squareLen^2 * 5/12}" iyz="0.0" izz="${armLink3squareLen^2 / 6}" />
 		</inertial>
 	</link>
@@ -210,4 +217,5 @@
 			<xacro:armLink4_geom />
 			<xacro:armLink4_offset />
+			<material name="blue"/>
 		</visual>
 		<collision>
@@ -217,5 +225,5 @@
 		<inertial>
 			<mass value="${armLink4Mass}" />
-			<inertia ixx="1.0" ixy="0.0" ixz="0.0" iyy="1.0" iyz="0.0" izz="1.0" />
+			<inertia ixx="${armLink4Len^2 /6}" ixy="0.0" ixz="0.0" iyy="${armLink4Len^2/6}" iyz="0.0" izz="${armLink4Len^2 /6}" />
 		</inertial>
 	</link>
@@ -242,4 +250,5 @@
 			<xacro:armLink5_geom />
 			<xacro:armLink5_offset />
+			<material name="white"/>
 		</visual>
 		<collision>
@@ -249,5 +258,5 @@
 		<inertial>
 			<mass value="${armLink5Mass}" />
-			<inertia ixx="1.0" ixy="0.0" ixz="0.0" iyy="1.0" iyz="0.0" izz="1.0" />
+			<inertia ixx="${armLink5Len^2/3+armLink5Rad^2/4}" ixy="0.0" ixz="0.0" iyy="${armLink5Len^2/3+armLink5Rad^2/4}" iyz="0.0" izz="${armLink5Rad^2/2}" />
 		</inertial>
 	</link>
@@ -272,4 +281,5 @@
 			<xacro:armLink5square_geom />
 			<xacro:armLink5square_offset />
+			<material name="white"/>
 		</visual>
 		<collision>
@@ -279,5 +289,5 @@
 		<inertial>
 			<mass value="${armLink5squareMass}" />
-			<inertia ixx="1.0" ixy="0.0" ixz="0.0" iyy="1.0" iyz="0.0" izz="1.0" />
+			<inertia ixx="${armLink5squareLen^2 * 5/12}" ixy="0.0" ixz="0.0" iyy="${armLink5squareLen^2 * 5/12}" iyz="0.0" izz="${armLink5squareLen^2 / 6}" />
 		</inertial>
 	</link>
@@ -301,4 +311,5 @@
 			<xacro:armLink6_geom />
 			<xacro:armLink6_offset />
+			<material name="blue"/>
 		</visual>
 		<collision>
@@ -308,5 +319,5 @@
 		<inertial>
 			<mass value="${armLink6Mass}" />
-			<inertia ixx="1.0" ixy="0.0" ixz="0.0" iyy="1.0" iyz="0.0" izz="1.0" />
+			<inertia ixx="${armLink6Len^2 /6}" ixy="0.0" ixz="0.0" iyy="${armLink6Len^2/6}" iyz="0.0" izz="${armLink6Len^2 /6}" />
 		</inertial>
 	</link>
@@ -333,4 +344,5 @@
 			<xacro:armLink7_geom />
 			<xacro:armLink7_offset />
+			<material name="white"/>
 		</visual>
 		<collision>
@@ -340,5 +352,5 @@
 		<inertial>
 			<mass value="${armLink7Mass}" />
-			<inertia ixx="1.0" ixy="0.0" ixz="0.0" iyy="1.0" iyz="0.0" izz="1.0" />
+			<inertia ixx="${armLink7Len^2/3+armLink7Rad^2/4}" ixy="0.0" ixz="0.0" iyy="${armLink7Len^2/3+armLink7Rad^2/4}" iyz="0.0" izz="${armLink7Rad^2/2}" />
 		</inertial>
 	</link>
@@ -363,4 +375,5 @@
 			<xacro:armLink7square_geom />
 			<xacro:armLink7square_offset />
+			<material name="white"/>
 		</visual>
 		<collision>
@@ -370,5 +383,5 @@
 		<inertial>
 			<mass value="${armLink7squareMass}" />
-			<inertia ixx="1.0" ixy="0.0" ixz="0.0" iyy="1.0" iyz="0.0" izz="1.0" />
+			<inertia ixx="${armLink7squareLen^2 * 5/12}" ixy="0.0" ixz="0.0" iyy="${armLink7squareLen^2 * 5/12}" iyz="0.0" izz="${armLink7squareLen^2 / 6}" />
 		</inertial>
 	</link>

Commit message: Readjusted sizes of links

File: src/urdf/restorebot.urdf.xacro (robot description, xacro)
@@ -55,5 +55,5 @@
 		</xacro:macro>
 		<xacro:property name="armLink1Rad" value="${cylRad}" />
-		<xacro:property name="armLink1Len" value = "${cylLen/4}" />
+		<xacro:property name="armLink1Len" value = "${cylLen/2}" />
 		<xacro:property name="armLink1Mass" value =
 				"${AlDensity*3.14*armLink1Len*armLink1Rad^2}" />
@@ -79,5 +79,5 @@
 	</joint>
 	<link name="armLink1square">
-		<xacro:property name="armLink1squareLen" value="${armLink1Rad}" />
+		<xacro:property name="armLink1squareLen" value="${armLink1Rad*2.2}" />
 		<xacro:property name="armLink1squareMass" value="${AlDensity*armLink1squareLen^3}" />
 		<xacro:macro name="armLink1square_geom">
@@ -174,5 +174,5 @@
 	</joint>
 	<link name="armLink3square">
-		<xacro:property name="armLink3squareLen" value="${armLink3Rad}" />
+		<xacro:property name="armLink3squareLen" value="${armLink3Rad*2.2}" />
 		<xacro:property name="armLink3squareMass" value="${AlDensity*armLink3squareLen^3}" />
 		<xacro:macro name="armLink3square_geom">
@@ -268,5 +268,5 @@
 	</joint>
 	<link name="armLink5square">
-		<xacro:property name="armLink5squareLen" value="${armLink5Rad}" />
+		<xacro:property name="armLink5squareLen" value="${armLink5Rad*2.2}" />
 		<xacro:property name="armLink5squareMass" value="${AlDensity*armLink5squareLen^3}" />
 		<xacro:macro name="armLink5square_geom">

Commit message: Added Satellite, Supports, and Comment Descriptions

File: src/urdf/restorebot.urdf.xacro (robot description, xacro)
@@ -2,33 +2,37 @@
 <robot name="restorebot" xmlns:xacro="http://ros.org/wiki/xacro">
 	<xacro:property name="AlDensity" value="2712" />
-	<xacro:property name="platLen" value="2" />
-	<xacro:property name="platWidth" value="2" />
+	<xacro:property name="platLen" value="8" />
+	<xacro:property name="platWidth" value="8" />
 	<xacro:property name="platHeight" value="1" />
-	<xacro:property name="box_mass" value="${AlDensity*platLen*platWidth*platHeight}" />
-	<xacro:macro name="default_box_inertia" params="mass">
-		<inertial>
-			<mass value="${mass}" />
-			<inertia ixx="1.0" ixy="0.0" ixz="0.0" iyy="1.0" iyz="0.0" izz="1.0" />
-		</inertial>
-	</xacro:macro>
+	<xacro:property name="satLen" value="${5}" />
+	<xacro:property name="satWidth" value="${5}" />
+	<xacro:property name="satHeight" value="${5}" />
 	<xacro:property name="cylRad" value="0.2" />
 	<xacro:property name="cylLen" value = "0.8" />
-	<xacro:property name="cyl_mass" value = "2" />
-	<xacro:macro name="default_cyl_inertia" params="mass">
-		<inertial>
-			<mass value="${mass}" />
-			<inertia ixx="1.0" ixy="0.0" ixz="0.0" iyy="1.0" iyz="0.0" izz="1.0" />
-		</inertial>
-	</xacro:macro>
 	<material name="blue">
 		<color rgba="0 0 0.8 1"/>
 	</material>
 	<material name="black">
-		<color rgba="0 0 0 1"/>
+		<color rgba="0 .2 0 1"/>
 	</material>
 	<material name="white">
 			<color rgba="1 1 1 1"/>
 	</material>
+	<!--	****************
+			****************
+			****************
+			Base Platform
+			****************
+			****************
+			****************
+	-->
 	<link name="platform_base">
+		<xacro:property name="box_mass" value="${AlDensity*platLen*platWidth*platHeight}" />
+		<xacro:macro name="default_box_inertia" params="mass">
+			<inertial>
+				<mass value="${mass}" />
+				<inertia ixx="${platHeight^2/12+platWidth^2/12}" ixy="0.0" ixz="0.0" iyy="${platHeight^2/12+platLen^2/12}" iyz="0.0" izz="${platLen^2/12 +platWidth^2/12}" />
+			</inertial>
+		</xacro:macro>
 		<xacro:macro name="platform_geom">
 			<geometry>
@@ -45,4 +49,12 @@
 		<xacro:default_box_inertia mass ="${box_mass}" />
 	</link>
+	<!--	****************
+			****************
+			****************
+ 				Arm Link 1
+			****************
+			****************
+			****************
+	-->
 	<link name="armLink1">
 		<xacro:macro name="armLink1_geom">
@@ -75,5 +87,5 @@
 		<parent link="platform_base"/>
 		<child link="armLink1"/>
-		<origin rpy = "0 0 0" xyz="0 0 ${platHeight/2}" />
+		<origin rpy = "0 0 0" xyz="${platLen/4} 0 ${platHeight/2}" />
 		<axis xyz = "0 0 1" />
 	</joint>
@@ -109,4 +121,12 @@
 		<origin rpy = "0 0 0" xyz="0 0 ${armLink1Len}" />
 	</joint>
+	<!--	****************
+			****************
+			****************
+ 				Arm Link 2
+			****************
+			****************
+			****************
+	-->
 	<link name="armLink2">
 		<xacro:property name="armLink2Len" value="${armLink1squareLen}" />
@@ -140,4 +160,12 @@
 		<axis xyz = "1 0 0" />
 	</joint>
+	<!--	****************
+			****************
+			****************
+ 				Arm Link 3
+			****************
+			****************
+			****************
+	-->
 	<link name="armLink3">
 		<xacro:macro name="armLink3_geom">
@@ -203,4 +231,12 @@
 		<origin rpy = "0 0 0" xyz="0 0 ${armLink3Len}" />
 	</joint>
+	<!--	****************
+			****************
+			****************
+ 				Arm Link 4
+			****************
+			****************
+			****************
+	-->
 	<link name="armLink4">
 		<xacro:property name="armLink4Len" value="${armLink3squareLen}" />
@@ -234,4 +270,12 @@
 		<axis xyz = "1 0 0" />
 	</joint>
+	<!--	****************
+			****************
+			****************
+ 				Arm Link 5
+			****************
+			****************
+			****************
+	-->
 	<link name="armLink5">
 		<xacro:macro name="armLink5_geom">
@@ -297,4 +341,12 @@
 		<origin rpy = "0 0 0" xyz="0 0 ${armLink5Len}" />
 	</joint>
+	<!--	****************
+			****************
+			****************
+ 				Arm Link 6
+			****************
+			****************
+			****************
+	-->
 	<link name="armLink6">
 		<xacro:property name="armLink6Len" value="${armLink5squareLen}" />
@@ -328,4 +380,12 @@
 		<axis xyz = "1 0 0" />
 	</joint>
+	<!--	****************
+			****************
+			****************
+ 				Arm Link 7
+			****************
+			****************
+			****************
+	-->
 	<link name="armLink7">
 		<xacro:macro name="armLink7_geom">
@@ -391,3 +451,127 @@
 		<origin rpy = "0 0 0" xyz="0 0 ${armLink7Len}" />
 	</joint>
+	<!--	****************
+			****************
+			****************
+ Beginning of the Satellite/Support Section
+			****************
+			****************
+			****************
+	-->
+	<xacro:property name="supArc" value="1" />
+	<xacro:property name="supLen" value=".6" />
+	<xacro:property name="supRad" value=".2" />
+	<xacro:property name="supMass" value =
+				"${AlDensity*3.14*supLen*supRad^2}" />
+	<xacro:macro name="sup_geom">
+		<geometry>
+			<cylinder length="${supLen}" radius="${supRad}"/>
+		</geometry>
+	</xacro:macro>
+	<link name = "support1">
+		<xacro:macro name="support1_offset">
+			<origin rpy = "0 0 0" xyz = "0 0 ${supLen/2}" />
+		</xacro:macro>
+		<visual>
+			<xacro:sup_geom />
+			<xacro:support1_offset />
+			<material name="black"/>
+		</visual>
+		<collision>
+			<xacro:sup_geom />
+			<xacro:support1_offset />
+		</collision>
+		<inertial>
+			<mass value="${supMass}" />
+			<inertia ixx="${supLen^2/3+supRad^2/4}" ixy="0.0" ixz="0.0" iyy="${supLen^2/3+supRad^2/4}" iyz="0.0" izz="${supRad^2/2}" />
+		</inertial>
+	</link>
+	<joint name="base_to_sup1" type ="fixed">
+		<parent link="platform_base"/>
+		<child link="support1"/>
+		<origin rpy = "0 0 0" xyz="${-1*platLen/4} ${-1*supArc} ${platHeight/2}" />
+	</joint>
+	<link name = "support2">
+		<xacro:macro name="support2_offset">
+			<origin rpy = "0 0 0" xyz = "0 0 ${supLen/2}" />
+		</xacro:macro>
+		<visual>
+			<xacro:sup_geom />
+			<xacro:support1_offset />
+			<material name="black"/>
+		</visual>
+		<collision>
+			<xacro:sup_geom />
+			<xacro:support1_offset />
+		</collision>
+		<inertial>
+			<mass value="${supMass}" />
+			<inertia ixx="${supLen^2/3+supRad^2/4}" ixy="0.0" ixz="0.0" iyy="${supLen^2/3+supRad^2/4}" iyz="0.0" izz="${supRad^2/2}" />
+		</inertial>
+	</link>
+	<joint name="base_to_sup2" type ="fixed">
+		<parent link="platform_base"/>
+		<child link="support2"/>
+		<origin rpy = "0 0 0" xyz="${-1*platLen/4+supArc*1.7/2} ${supArc/2} ${platHeight/2}" />
+	</joint>
+	<link name = "support3">
+		<xacro:macro name="support3_offset">
+			<origin rpy = "0 0 0" xyz = "0 0 ${supLen/2}" />
+		</xacro:macro>
+		<visual>
+			<xacro:sup_geom />
+			<xacro:support1_offset />
+			<material name="black"/>
+		</visual>
+		<collision>
+			<xacro:sup_geom />
+			<xacro:support1_offset />
+		</collision>
+		<inertial>
+			<mass value="${supMass}" />
+			<inertia ixx="${supLen^2/3+supRad^2/4}" ixy="0.0" ixz="0.0" iyy="${supLen^2/3+supRad^2/4}" iyz="0.0" izz="${supRad^2/2}" />
+		</inertial>
+	</link>
+	<joint name="base_to_sup3" type ="fixed">
+		<parent link="platform_base"/>
+		<child link="support3"/>
+		<origin rpy = "0 0 0" xyz="${-1*platLen/4-supArc*1.7/2} ${supArc/2} ${platHeight/2}" />
+	</joint>
+	<!--	****************
+			****************
+			****************
+	 			Satellite
+			****************
+			****************
+			****************
+	-->
+	<link name="satellite">
+		<xacro:property name="satMass" value="${AlDensity*satLen*satWidth*satHeight}" />
+		<xacro:macro name="sat_geom">
+			<geometry>
+				<box size="${satLen} ${satWidth} ${satHeight}"/>
+			</geometry>
+		</xacro:macro>
+		<xacro:macro name="sat_offset">
+			<origin rpy = "0 0 0" xyz="0 0 ${satHeight/2}" />
+		</xacro:macro>
+		<visual>
+			<xacro:sat_geom />
+			<xacro:sat_offset />
+			<material name="black"/>
+		</visual>
+		<collision>
+			<xacro:sat_geom />
+			<xacro:sat_offset />
+		</collision>
+		<inertial>
+			<mass value="${satMass}" />
+			<inertia ixx="${satHeight^2/3+satWidth^2/12}" ixy="0.0" ixz="0.0" iyy="${satHeight^2/3+satLen^2/12}" iyz="0.0" izz="${satLen^2/12 +satWidth^2/12}" />
+		</inertial>
+	</link>
+	<joint name="sup1_to_satellite" type ="fixed">
+		<parent link="support1"/>
+		<child link="satellite"/>
+		<origin rpy = "0 0 0" xyz="${0} ${supArc} ${supLen}" />
+	</joint>
 </robot>
