Commit message: Fixed Exponential Math and Updated to Kinetic

File: src/urdf/restorebot.urdf.xacro (robot description, xacro)
@@ -32,5 +32,5 @@
 			<inertial>
 				<mass value="${mass}" />
-				<inertia ixx="${platHeight^2/12+platWidth^2/12}" ixy="0.0" ixz="0.0" iyy="${platHeight^2/12+platLen^2/12}" iyz="0.0" izz="${platLen^2/12 +platWidth^2/12}" />
+				<inertia ixx="${platHeight*platHeight/12+platWidth*platWidth/12}" ixy="0.0" ixz="0.0" iyy="${platHeight*platHeight/12+platLen*platLen/12}" iyz="0.0" izz="${platLen*platLen/12 +platWidth*platWidth/12}" />
 			</inertial>
 		</xacro:macro>
@@ -69,5 +69,5 @@
 		<xacro:property name="armLink1Len" value = "${cylLen/2}" />
 		<xacro:property name="armLink1Mass" value =
-				"${AlDensity*3.14*armLink1Len*armLink1Rad^2}" />
+				"${AlDensity*3.14*armLink1Len*armLink1Rad*armLink1Rad}" />
 		<visual>
 			<xacro:armLink1_geom />
@@ -81,5 +81,5 @@
 		<inertial>
 			<mass value="${armLink1Mass}" />
-			<inertia ixx="${armLink1Len^2/3+armLink1Rad^2/4}" ixy="0.0" ixz="0.0" iyy="${armLink1Len^2/3+armLink1Rad^2/4}" iyz="0.0" izz="${armLink1Rad^2/2}" />
+			<inertia ixx="${armLink1Len*armLink1Len/3+armLink1Rad*armLink1Rad/4}" ixy="0.0" ixz="0.0" iyy="${armLink1Len*armLink1Len/3+armLink1Rad*armLink1Rad/4}" iyz="0.0" izz="${armLink1Rad*armLink1Rad/2}" />
 		</inertial>
 	</link>
@@ -92,5 +92,5 @@
 	<link name="armLink1square">
 		<xacro:property name="armLink1squareLen" value="${armLink1Rad*2.2}" />
-		<xacro:property name="armLink1squareMass" value="${AlDensity*armLink1squareLen^3}" />
+		<xacro:property name="armLink1squareMass" value="${AlDensity*armLink1squareLen*armLink1squareLen*armLink1squareLen}" />
 		<xacro:macro name="armLink1square_geom">
 			<geometry>
@@ -112,5 +112,5 @@
 		<inertial>
 			<mass value="${armLink1squareMass}" />
-			<inertia ixx="${armLink1squareLen^2 * 5/12}" ixy="0.0" ixz="0.0" iyy="${armLink1squareLen^2 * 5/12}" iyz="0.0" izz="${armLink1squareLen^2 / 6}" />
+			<inertia ixx="${armLink1squareLen*armLink1squareLen * 5/12}" ixy="0.0" ixz="0.0" iyy="${armLink1squareLen*armLink1squareLen * 5/12}" iyz="0.0" izz="${armLink1squareLen*armLink1squareLen / 6}" />
 		</inertial>
 	</link>
@@ -131,5 +131,5 @@
 	<link name="armLink2">
 		<xacro:property name="armLink2Len" value="${armLink1squareLen}" />
-		<xacro:property name="armLink2Mass" value="${AlDensity*armLink2Len^3}" />
+		<xacro:property name="armLink2Mass" value="${AlDensity*armLink2Len*armLink2Len*armLink2Len}" />
 		<xacro:macro name="armLink2_geom">
 			<geometry>
@@ -151,5 +151,5 @@
 		<inertial>
 			<mass value="${armLink2Mass}" />
-			<inertia ixx="${armLink2Len^2 /6}" ixy="0.0" ixz="0.0" iyy="${armLink2Len^2/6}" iyz="0.0" izz="${armLink2Len^2 /6}" />
+			<inertia ixx="${armLink2Len*armLink2Len /6}" ixy="0.0" ixz="0.0" iyy="${armLink2Len*armLink2Len/6}" iyz="0.0" izz="${armLink2Len*armLink2Len /6}" />
 		</inertial>
 	</link>
@@ -180,5 +180,5 @@
 		<xacro:property name="armLink3Len" value = "${cylLen}" />
 		<xacro:property name="armLink3Mass" value =
-				"${AlDensity*3.14*armLink3Len*armLink3Rad^2}" />
+				"${AlDensity*3.14*armLink3Len*armLink3Rad*armLink3Rad}" />
 		<visual>
 			<xacro:armLink3_geom />
@@ -192,5 +192,5 @@
 		<inertial>
 			<mass value="${armLink3Mass}" />
-			<inertia ixx="${armLink3Len^2/3+armLink3Rad^2/4}" ixy="0.0" ixz="0.0" iyy="${armLink3Len^2/3+armLink3Rad^2/4}" iyz="0.0" izz="${armLink3Rad^2/2}" />
+			<inertia ixx="${armLink3Len*armLink3Len/3+armLink3Rad*armLink3Rad/4}" ixy="0.0" ixz="0.0" iyy="${armLink3Len*armLink3Len/3+armLink3Rad*armLink3Rad/4}" iyz="0.0" izz="${armLink3Rad*armLink3Rad/2}" />
 		</inertial>
 	</link>
@@ -203,5 +203,5 @@
 	<link name="armLink3square">
 		<xacro:property name="armLink3squareLen" value="${armLink3Rad*2.2}" />
-		<xacro:property name="armLink3squareMass" value="${AlDensity*armLink3squareLen^3}" />
+		<xacro:property name="armLink3squareMass" value="${AlDensity*armLink3squareLen*armLink3squareLen*armLink3squareLen}" />
 		<xacro:macro name="armLink3square_geom">
 			<geometry>
@@ -223,5 +223,5 @@
 		<inertial>
 			<mass value="${armLink3squareMass}" />
-			<inertia ixx="${armLink3squareLen^2 * 5/12}" ixy="0.0" ixz="0.0" iyy="${armLink3squareLen^2 * 5/12}" iyz="0.0" izz="${armLink3squareLen^2 / 6}" />
+			<inertia ixx="${armLink3squareLen*armLink3squareLen * 5/12}" ixy="0.0" ixz="0.0" iyy="${armLink3squareLen*armLink3squareLen * 5/12}" iyz="0.0" izz="${armLink3squareLen*armLink3squareLen / 6}" />
 		</inertial>
 	</link>
@@ -241,5 +241,5 @@
 	<link name="armLink4">
 		<xacro:property name="armLink4Len" value="${armLink3squareLen}" />
-		<xacro:property name="armLink4Mass" value="${AlDensity*armLink4Len^3}" />
+		<xacro:property name="armLink4Mass" value="${AlDensity*armLink4Len*armLink4Len*armLink4Len}" />
 		<xacro:macro name="armLink4_geom">
 			<geometry>
@@ -261,5 +261,5 @@
 		<inertial>
 			<mass value="${armLink4Mass}" />
-			<inertia ixx="${armLink4Len^2 /6}" ixy="0.0" ixz="0.0" iyy="${armLink4Len^2/6}" iyz="0.0" izz="${armLink4Len^2 /6}" />
+			<inertia ixx="${armLink4Len*armLink4Len /6}" ixy="0.0" ixz="0.0" iyy="${armLink4Len*armLink4Len/6}" iyz="0.0" izz="${armLink4Len*armLink4Len /6}" />
 		</inertial>
 	</link>
@@ -290,5 +290,5 @@
 		<xacro:property name="armLink5Len" value = "${cylLen}" />
 		<xacro:property name="armLink5Mass" value =
-				"${AlDensity*3.14*armLink5Len*armLink5Rad^2}" />
+				"${AlDensity*3.14*armLink5Len*armLink5Rad*armLink5Rad}" />
 		<visual>
 			<xacro:armLink5_geom />
@@ -302,5 +302,5 @@
 		<inertial>
 			<mass value="${armLink5Mass}" />
-			<inertia ixx="${armLink5Len^2/3+armLink5Rad^2/4}" ixy="0.0" ixz="0.0" iyy="${armLink5Len^2/3+armLink5Rad^2/4}" iyz="0.0" izz="${armLink5Rad^2/2}" />
+			<inertia ixx="${armLink5Len*armLink5Len/3+armLink5Rad*armLink5Rad/4}" ixy="0.0" ixz="0.0" iyy="${armLink5Len*armLink5Len/3+armLink5Rad*armLink5Rad/4}" iyz="0.0" izz="${armLink5Rad*armLink5Rad/2}" />
 		</inertial>
 	</link>
@@ -313,5 +313,5 @@
 	<link name="armLink5square">
 		<xacro:property name="armLink5squareLen" value="${armLink5Rad*2.2}" />
-		<xacro:property name="armLink5squareMass" value="${AlDensity*armLink5squareLen^3}" />
+		<xacro:property name="armLink5squareMass" value="${AlDensity*armLink5squareLen*armLink5squareLen*armLink5squareLen}" />
 		<xacro:macro name="armLink5square_geom">
 			<geometry>
@@ -333,5 +333,5 @@
 		<inertial>
 			<mass value="${armLink5squareMass}" />
-			<inertia ixx="${armLink5squareLen^2 * 5/12}" ixy="0.0" ixz="0.0" iyy="${armLink5squareLen^2 * 5/12}" iyz="0.0" izz="${armLink5squareLen^2 / 6}" />
+			<inertia ixx="${armLink5squareLen*armLink5squareLen * 5/12}" ixy="0.0" ixz="0.0" iyy="${armLink5squareLen*armLink5squareLen * 5/12}" iyz="0.0" izz="${armLink5squareLen*armLink5squareLen / 6}" />
 		</inertial>
 	</link>
@@ -351,5 +351,5 @@
 	<link name="armLink6">
 		<xacro:property name="armLink6Len" value="${armLink5squareLen}" />
-		<xacro:property name="armLink6Mass" value="${AlDensity*armLink6Len^3}" />
+		<xacro:property name="armLink6Mass" value="${AlDensity*armLink6Len*armLink6Len*armLink6Len}" />
 		<xacro:macro name="armLink6_geom">
 			<geometry>
@@ -371,5 +371,5 @@
 		<inertial>
 			<mass value="${armLink6Mass}" />
-			<inertia ixx="${armLink6Len^2 /6}" ixy="0.0" ixz="0.0" iyy="${armLink6Len^2/6}" iyz="0.0" izz="${armLink6Len^2 /6}" />
+			<inertia ixx="${armLink6Len*armLink6Len /6}" ixy="0.0" ixz="0.0" iyy="${armLink6Len*armLink6Len/6}" iyz="0.0" izz="${armLink6Len*armLink6Len /6}" />
 		</inertial>
 	</link>
@@ -400,5 +400,5 @@
 		<xacro:property name="armLink7Len" value = "${armLink1Len}" />
 		<xacro:property name="armLink7Mass" value =
-				"${AlDensity*3.14*armLink7Len*armLink7Rad^2}" />
+				"${AlDensity*3.14*armLink7Len*armLink7Rad*armLink7Rad}" />
 		<visual>
 			<xacro:armLink7_geom />
@@ -412,5 +412,5 @@
 		<inertial>
 			<mass value="${armLink7Mass}" />
-			<inertia ixx="${armLink7Len^2/3+armLink7Rad^2/4}" ixy="0.0" ixz="0.0" iyy="${armLink7Len^2/3+armLink7Rad^2/4}" iyz="0.0" izz="${armLink7Rad^2/2}" />
+			<inertia ixx="${armLink7Len*armLink7Len/3+armLink7Rad*armLink7Rad/4}" ixy="0.0" ixz="0.0" iyy="${armLink7Len*armLink7Len/3+armLink7Rad*armLink7Rad/4}" iyz="0.0" izz="${armLink7Rad*armLink7Rad/2}" />
 		</inertial>
 	</link>
@@ -423,5 +423,5 @@
 	<link name="armLink7square">
 		<xacro:property name="armLink7squareLen" value="${armLink7Rad}" />
-		<xacro:property name="armLink7squareMass" value="${AlDensity*armLink7squareLen^3}" />
+		<xacro:property name="armLink7squareMass" value="${AlDensity*armLink7squareLen*armLink7squareLen*armLink7squareLen}" />
 		<xacro:macro name="armLink7square_geom">
 			<geometry>
@@ -443,5 +443,5 @@
 		<inertial>
 			<mass value="${armLink7squareMass}" />
-			<inertia ixx="${armLink7squareLen^2 * 5/12}" ixy="0.0" ixz="0.0" iyy="${armLink7squareLen^2 * 5/12}" iyz="0.0" izz="${armLink7squareLen^2 / 6}" />
+			<inertia ixx="${armLink7squareLen*armLink7squareLen * 5/12}" ixy="0.0" ixz="0.0" iyy="${armLink7squareLen*armLink7squareLen * 5/12}" iyz="0.0" izz="${armLink7squareLen*armLink7squareLen / 6}" />
 		</inertial>
 	</link>
@@ -463,5 +463,5 @@
 	<xacro:property name="supRad" value=".2" />
 	<xacro:property name="supMass" value =
-				"${AlDensity*3.14*supLen*supRad^2}" />
+				"${AlDensity*3.14*supLen*supRad*supRad}" />
 	<xacro:macro name="sup_geom">
 		<geometry>
@@ -469,4 +469,10 @@
 		</geometry>
 	</xacro:macro>
+	<xacro:macro name="sup_inertia">
+		<inertial>
+			<mass value="${supMass}" />
+			<inertia ixx="${supLen*supLen/3+supRad*supRad/4}" ixy="0.0" ixz="0.0" iyy="${supLen*supLen/3+supRad*supRad/4}" iyz="0.0" izz="${supRad*supRad/2}" />
+		</inertial>
+	</xacro:macro>
 	<link name = "support1">
 		<xacro:macro name="support1_offset">
@@ -482,8 +488,5 @@
 			<xacro:support1_offset />
 		</collision>
-		<inertial>
-			<mass value="${supMass}" />
-			<inertia ixx="${supLen^2/3+supRad^2/4}" ixy="0.0" ixz="0.0" iyy="${supLen^2/3+supRad^2/4}" iyz="0.0" izz="${supRad^2/2}" />
-		</inertial>
+		<xacro:sup_inertia />
 	</link>
 	<joint name="base_to_sup1" type ="fixed">
@@ -505,8 +508,5 @@
 			<xacro:support1_offset />
 		</collision>
-		<inertial>
-			<mass value="${supMass}" />
-			<inertia ixx="${supLen^2/3+supRad^2/4}" ixy="0.0" ixz="0.0" iyy="${supLen^2/3+supRad^2/4}" iyz="0.0" izz="${supRad^2/2}" />
-		</inertial>
+		<xacro:sup_inertia />
 	</link>
 	<joint name="base_to_sup2" type ="fixed">
@@ -528,8 +528,5 @@
 			<xacro:support1_offset />
 		</collision>
-		<inertial>
-			<mass value="${supMass}" />
-			<inertia ixx="${supLen^2/3+supRad^2/4}" ixy="0.0" ixz="0.0" iyy="${supLen^2/3+supRad^2/4}" iyz="0.0" izz="${supRad^2/2}" />
-		</inertial>
+		<xacro:sup_inertia />
 	</link>
 	<joint name="base_to_sup3" type ="fixed">
@@ -567,6 +564,6 @@
 		<inertial>
 			<mass value="${satMass}" />
-			<inertia ixx="${satHeight^2/3+satWidth^2/12}" ixy="0.0" ixz="0.0" iyy="${satHeight^2/3+satLen^2/12}" iyz="0.0" izz="${satLen^2/12 +satWidth^2/12}" />
-		</inertial>
+			<inertia ixx="${satHeight*satHeight/3+satWidth*satWidth/12}" ixy="0.0" ixz="0.0" iyy="${satHeight*satHeight/3+satLen*satLen/12}" iyz="0.0" izz="${satLen*satLen/12 +satWidth*satWidth/12}" />
+</inertial>
 	</link>
 	<joint name="sup1_to_satellite" type ="fixed">
@@ -575,3 +572,4 @@
 		<origin rpy = "0 0 0" xyz="${0} ${supArc} ${supLen}" />
 	</joint>
+n
 </robot>
