Commit message: Updated Clutter

File: src/urdf/restorebot.urdf (robot description, URDF)
Before this commit: robot restorebot, 12 links, 11 joints
Links:
- added link clutter1, mass 73.224; collision sphere radius=0.3; visual sphere radius=0.3
- added link clutter2, mass 21.696; collision sphere radius=0.2; visual sphere radius=0.2
- added link satellite, mass 339000; collision box size=5 5 5; visual box size=5 5 5
- added link support1, mass 510.9408; collision cylinder length=1.5 radius=0.2; visual cylinder length=1.5 radius=0.2
- added link support2, mass 510.9408; collision cylinder length=1.5 radius=0.2; visual cylinder length=1.5 radius=0.2
- added link support3, mass 510.9408; collision cylinder length=1.5 radius=0.2; visual cylinder length=1.5 radius=0.2
- link armLink1: mass 340.6272 -> 136.25088; geometry collision cylinder length=0.4 radius=0.2; visual cylinder length=0.4 radius=0.2
- link armLink1square: mass 542.4 -> 231.019008; geometry collision box size=0.44 0.44 0.44; visual box size=0.44 0.44 0.44
- link armLink2: mass 542.4 -> 231.019008; geometry collision box size=0.44 0.44 0.44; visual box size=0.44 0.44 0.44
- link armLink3: mass 1362.5088 -> 272.50176
- link armLink3square: mass 542.4 -> 231.019008; geometry collision box size=0.44 0.44 0.44; visual box size=0.44 0.44 0.44
- link armLink4: mass 542.4 -> 231.019008; geometry collision box size=0.44 0.44 0.44; visual box size=0.44 0.44 0.44
- link armLink5: mass 1362.5088 -> 272.50176
- link armLink5square: mass 542.4 -> 231.019008; geometry collision box size=0.44 0.44 0.44; visual box size=0.44 0.44 0.44
- link armLink6: mass 542.4 -> 231.019008; geometry collision box size=0.44 0.44 0.44; visual box size=0.44 0.44 0.44
- link armLink7: mass 340.6272 -> 136.25088; geometry collision cylinder length=0.4 radius=0.2; visual cylinder length=0.4 radius=0.2
- link armLink7square: mass 542.4 -> 21.696
- link platform_base: mass 10848.0 -> 173568; geometry collision box size=8 8 1; visual box size=8 8 1
Joints:
- added joint base_to_sup1: type fixed, parent platform_base, child support1, origin xyz=-2.0 -1 0.5 rpy=0 0 0
- added joint base_to_sup2: type fixed, parent platform_base, child support2, origin xyz=-1.15 0.5 0.5 rpy=0 0 0
- added joint base_to_sup3: type fixed, parent platform_base, child support3, origin xyz=-2.85 0.5 0.5 rpy=0 0 0
- added joint platform_to_clutter1: type fixed, parent platform_base, child clutter1, origin xyz=2 2 3 rpy=0 0 0
- added joint platform_to_clutter2: type fixed, parent platform_base, child clutter2, origin xyz=1.5 0 2 rpy=0 0 0
- added joint sup1_to_satellite: type fixed, parent support1, child satellite, origin xyz=0 1 1.5 rpy=0 0 0
- joint armLink1Fixed: origin xyz=0 0 0.2 rpy=0 0 0 -> xyz=0 0 0.4 rpy=0 0 0
- joint armLink1_to_armLink2: origin xyz=0.2 0 0.1 rpy=0 0 0 -> xyz=0.44 0 0.22 rpy=0 0 0
- joint armLink2_to_armLink3: origin xyz=0 0 0.1 rpy=0 0 0 -> xyz=0 0 0.22 rpy=0 0 0
- joint armLink3_to_armLink4: origin xyz=0.2 0 0.1 rpy=0 0 0 -> xyz=0.44 0 0.22 rpy=0 0 0
- joint armLink4_to_armLink5: origin xyz=0 0 0.1 rpy=0 0 0 -> xyz=0 0 0.22 rpy=0 0 0
- joint armLink5_to_armLink6: origin xyz=-0.2 0 0.1 rpy=0 0 0 -> xyz=-0.44 0 0.22 rpy=0 0 0
- joint armLink6_to_armLink7: origin xyz=0 0 0.1 rpy=0 0 0 -> xyz=0 0 0.22 rpy=0 0 0
- joint armLink7Fixed: origin xyz=0 0 0.2 rpy=0 0 0 -> xyz=0 0 0.4 rpy=0 0 0
- joint base_to_link1: origin xyz=0 0 0.5 rpy=0 0 0 -> xyz=2.0 2.0 0.5 rpy=0 0 0

File: src/urdf/restorebot.urdf.xacro (robot description, xacro)
@@ -17,5 +17,8 @@
 	</material>
 	<material name="white">
-			<color rgba="1 1 1 1"/>
+		<color rgba="1 1 1 1"/>
+	</material>
+	<material name="cyan">
+		<color rgba="0 1 1 1"/>
 	</material>
 	<!--	****************
@@ -87,5 +90,5 @@
 		<parent link="platform_base"/>
 		<child link="armLink1"/>
-		<origin rpy = "0 0 0" xyz="${platLen/4} 0 ${platHeight/2}" />
+		<origin rpy = "0 0 0" xyz="${platLen/4} ${platWidth/4} ${platHeight/2}" />
 		<axis xyz = "0 0 1" />
 	</joint>
@@ -460,5 +463,5 @@
 	-->
 	<xacro:property name="supArc" value="1" />
-	<xacro:property name="supLen" value=".6" />
+	<xacro:property name="supLen" value="1.5" />
 	<xacro:property name="supRad" value=".2" />
 	<xacro:property name="supMass" value =
@@ -564,6 +567,6 @@
 		<inertial>
 			<mass value="${satMass}" />
-			<inertia ixx="${satHeight*satHeight/3+satWidth*satWidth/12}" ixy="0.0" ixz="0.0" iyy="${satHeight*satHeight/3+satLen*satLen/12}" iyz="0.0" izz="${satLen*satLen/12 +satWidth*satWidth/12}" />
-</inertial>
+			<inertia ixx="${satHeight*satHeight/3+satWidth*satWidth/12}" ixy="0.0" ixz="0.0" iyy="${satHeight*satHeight/3+satLen*satLen/12}" iyz="0.0" izz="${satLen*satLen/+satWidth*satWidth/12}" />
+		</inertial>
 	</link>
 	<joint name="sup1_to_satellite" type ="fixed">
@@ -572,4 +575,61 @@
 		<origin rpy = "0 0 0" xyz="${0} ${supArc} ${supLen}" />
 	</joint>
-n
+	<!--	****************
+			****************
+			****************
+	 		  Clutter
+			****************
+			****************
+			****************
+	-->
+	<link name="clutter1">
+		<xacro:property name="c1Mass" value="${AlDensity*c1Rad*c1Rad*c1Rad}" />
+		<xacro:property name="c1Rad" value=".3" />
+		<xacro:macro name="c1_geom">
+			<geometry>
+				<sphere radius="${c1Rad}"/>
+			</geometry>
+		</xacro:macro>
+		<visual>
+			<xacro:c1_geom />
+			<material name="cyan"/>
+		</visual>
+		<collision>
+			<xacro:c1_geom />
+		</collision>
+		<inertial>
+			<mass value="${c1Mass}" />
+			<inertia ixx="${2/5*c1Rad*c1Rad}" ixy="0.0" ixz="0.0" iyy="${2/5*c1Rad*c1Rad}" iyz="0.0" izz="${2/5*c1Rad*c1Rad}" />
+		</inertial>
+	</link>
+	<joint name="platform_to_clutter1" type="fixed">
+		<parent link="platform_base"/>
+		<child link="clutter1"/>
+		<origin rpy = "0 0 0" xyz = "${2} ${2} ${platHeight+2}" />
+	</joint>
+	<link name="clutter2">
+		<xacro:property name="c2Mass" value="${AlDensity*c2Rad*c2Rad*c2Rad}" />
+		<xacro:property name="c2Rad" value=".2" />
+		<xacro:macro name="c2_geom">
+			<geometry>
+				<sphere radius="${c2Rad}"/>
+			</geometry>
+		</xacro:macro>
+		<visual>
+			<xacro:c2_geom />
+			<material name="cyan"/>
+		</visual>
+		<collision>
+			<xacro:c2_geom />
+		</collision>
+		<inertial>
+			<mass value="${c2Mass}" />
+			<inertia ixx="${2/5*c2Rad*c2Rad}" ixy="0.0" ixz="0.0" iyy="${2/5*c2Rad*c2Rad}" iyz="0.0" izz="${2/5*c2Rad*c2Rad}" />
+		</inertial>
+	</link>
+	<joint name="platform_to_clutter2" type="fixed">
+		<parent link="platform_base"/>
+		<child link="clutter2"/>
+		<origin rpy = "0 0 0" xyz = "${1.5} ${0} ${platHeight+1}" />
+	</joint>
 </robot>

Commit message: Updated to Revolute Joints to Fix Trajectory Problems

File: src/urdf/restorebot.urdf (robot description, URDF)
Before this commit: robot restorebot, 18 links, 17 joints
Joints:
- joint armLink1_to_armLink2: limit (none) -> lower=-3.14 upper=3.14 effort=100 velocity=3; type continuous -> revolute
- joint armLink2_to_armLink3: limit (none) -> lower=-3.14 upper=3.14 effort=100 velocity=3; type continuous -> revolute
- joint armLink3_to_armLink4: limit (none) -> lower=-3.14 upper=3.14 effort=100 velocity=3; type continuous -> revolute
- joint armLink4_to_armLink5: limit (none) -> lower=-3.14 upper=3.14 effort=100 velocity=3; type continuous -> revolute
- joint armLink5_to_armLink6: limit (none) -> lower=-3.14 upper=3.14 effort=100 velocity=3; type continuous -> revolute
- joint armLink6_to_armLink7: limit (none) -> lower=-3.14 upper=3.14 effort=100 velocity=3; type continuous -> revolute
- joint base_to_link1: limit (none) -> lower=-3.14 upper=3.14 effort=100 velocity=3; type continuous -> revolute

File: src/urdf/restorebot.urdf.xacro (robot description, xacro)
@@ -87,9 +87,10 @@
 		</inertial>
 	</link>
-	<joint name="base_to_link1" type ="continuous">
+	<joint name="base_to_link1" type ="revolute">
 		<parent link="platform_base"/>
 		<child link="armLink1"/>
 		<origin rpy = "0 0 0" xyz="${platLen/4} ${platWidth/4} ${platHeight/2}" />
 		<axis xyz = "0 0 1" />
+		<limit effort="100" lower="-3.14" upper="3.14" velocity="3"/>
 	</joint>
 	<link name="armLink1square">
@@ -157,9 +158,10 @@
 		</inertial>
 	</link>
-	<joint name="armLink1_to_armLink2" type ="continuous">
+	<joint name="armLink1_to_armLink2" type ="revolute">
 		<parent link="armLink1square"/>
 		<child link="armLink2"/>
 		<origin rpy = "0 0 0" xyz="${armLink1squareLen} 0 ${armLink2Len/2}" />
 		<axis xyz = "1 0 0" />
+		<limit effort="100" lower="-3.14" upper="3.14" velocity="3"/>
 	</joint>
 	<!--	****************
@@ -198,9 +200,10 @@
 		</inertial>
 	</link>
-	<joint name="armLink2_to_armLink3" type ="continuous">
+	<joint name="armLink2_to_armLink3" type ="revolute">
 		<parent link="armLink2"/>
 		<child link="armLink3"/>
 		<origin rpy = "0 0 0" xyz="0 0 ${armLink2Len/2}" />
 		<axis xyz = "0 0 1" />
+		<limit effort="100" lower="-3.14" upper="3.14" velocity="3"/>
 	</joint>
 	<link name="armLink3square">
@@ -267,9 +270,10 @@
 		</inertial>
 	</link>
-	<joint name="armLink3_to_armLink4" type ="continuous">
+	<joint name="armLink3_to_armLink4" type ="revolute">
 		<parent link="armLink3square"/>
 		<child link="armLink4"/>
 		<origin rpy = "0 0 0" xyz="${armLink3squareLen} 0 ${armLink4Len/2}" />
 		<axis xyz = "1 0 0" />
+		<limit effort="100" lower="-3.14" upper="3.14" velocity="3"/>
 	</joint>
 	<!--	****************
@@ -308,9 +312,10 @@
 		</inertial>
 	</link>
-	<joint name="armLink4_to_armLink5" type ="continuous">
+	<joint name="armLink4_to_armLink5" type ="revolute">
 		<parent link="armLink4"/>
 		<child link="armLink5"/>
 		<origin rpy = "0 0 0" xyz="0 0 ${armLink4Len/2}" />
 		<axis xyz = "0 0 1" />
+		<limit effort="100" lower="-3.14" upper="3.14" velocity="3"/>
 	</joint>
 	<link name="armLink5square">
@@ -377,9 +382,10 @@
 		</inertial>
 	</link>
-	<joint name="armLink5_to_armLink6" type ="continuous">
+	<joint name="armLink5_to_armLink6" type ="revolute">
 		<parent link="armLink5square"/>
 		<child link="armLink6"/>
 		<origin rpy = "0 0 0" xyz="${-1*armLink5squareLen} 0 ${armLink6Len/2}" />
 		<axis xyz = "1 0 0" />
+		<limit effort="100" lower="-3.14" upper="3.14" velocity="3"/>
 	</joint>
 	<!--	****************
@@ -418,9 +424,10 @@
 		</inertial>
 	</link>
-	<joint name="armLink6_to_armLink7" type ="continuous">
+	<joint name="armLink6_to_armLink7" type ="revolute">
 		<parent link="armLink6"/>
 		<child link="armLink7"/>
 		<origin rpy = "0 0 0" xyz="0 0 ${armLink6Len/2}" />
 		<axis xyz = "0 0 1" />
+		<limit effort="100" lower="-3.14" upper="3.14" velocity="3"/>
 	</joint>
 	<link name="armLink7square">
